File: AlarmConnector/AlarmConnector.sch (KiCad schematic (older format))
At the start: 23 parts, among them U1 LM393, U2 MT8870, U3 WeMos_mini

Commit message: update 1
Parts:
- removed C?: C, symbol C
- added C1: 100uF, symbol CP
- added C6, C9: 100nF, symbol C
- added C7, C8: 10nF, symbol C
- added R10, R11: 11k, symbol R
- added R12: 300k, symbol R
- added R13, R14, R6: 10k, symbol R
- added R8, R9: 100k, symbol R
- added U4: LM393, symbol LM393
- added Y1: 3.579547MHz, symbol Crystal
- C2: renamed from C?; value CP -> 10uF
- C3: renamed from C?; value CP -> 100uF
- C4, C5: renamed from C?; value C -> 100nF
- D2, D3: renamed from D?; value D_Zener -> 5V
- R1: renamed from R?; value R -> 2.2k
- R2: renamed from R?; value R -> 47k
- R3: renamed from R?; value R -> 10
- R4: renamed from R?; value R -> 15
- R5: renamed from R?; value R -> 1k
- R7: renamed from R?; value R -> 10k
- RV1: renamed from RV?; value POT -> 10k
- gave numbers to parts that had none: 6
Connections:
- net +5V: now also U2.10 (TOE), U2.18 (VDD), U3.1 (5V), C9.1, U4.8 (V+), U4.8 (V+)
- net GNDD: now also D2.1 (K), U2.9 (VSS), U3.2 (GND), C8.1, R14.1, R6.1, U4.4 (V-), U4.4 (V-)
- net at J1.2 (Pin_2), T1.2 (AB): now also C1.1
- net at Q2.1 (G): now also U3.4 (D3), R6.2
- net at R7.2, U1.1: now also U3.15 (D8)
- net at U2.1 (IN+): now also U2.4 (Vref)
- net at U2.11 (Q1): now also U3.6 (D1)
- net at U2.12 (Q2): now also U3.5 (D2)
- net at U2.13 (Q3): now also U3.13 (D6)
- net at U2.14 (Q4): now also U3.14 (D7)
- net at U2.15 (STD): now also U3.12 (D5)
- net at U2.16 (EST): now also R12.2
- net at U2.17 (ST/GT): now also C9.2, R12.1
- net at U2.2 (IN-): now also R8.1, R9.2
- net at U2.3 (GS): now also R9.1
- net at U2.7 (OSC1): now also Y1.1
- net at U2.8 (OSC2): now also Y1.2
- net at U3.3 (D4): now also R13.1
- net at D3.1 (K): now also C6.1, R8.2
- net at D3.2 (A): now also D2.2 (A)
- new net: C1.2, C6.2, C7.2, U4.1, U4.2 (_)
- new net: C8.2, R10.2, U4.3 (+)
- new net: R13.2, R14.2, U4.5 (+)
- new net: R11.1, U4.6 (_), U4.7
- new net: C7.1, R10.1, R11.2
Other:
- moved on the sheet: D2, D3, U3
